Commit message: fine tune robot model and update package.xml

File: urdf/mobile_robot_lidar.xacro (robot description, xacro)
@@ -2,5 +2,5 @@
 <robot xmlns:xacro="http://www.ros.org/wiki/xacro">
   <xacro:macro name="mobile_robot_lidar" params="prefix">
-    <!-- copy from robot macro -->
+    <!-- copied from robot macro -->
     <xacro:property name="bodylen" value="0.5461"/>
     <xacro:property name="lidarlen" value="0.1"/>
@@ -44,5 +44,5 @@
           <scan>
             <horizontal>
-              <samples>200</samples>
+              <samples>150</samples>
               <resolution>1</resolution>
               <min_angle>-1.570796</min_angle>
@@ -50,5 +50,5 @@
             </horizontal>
           </scan>
-          <resolution>0.001</resolution>
+          <!-- <resolution>0.001</resolution> -->
           <range>
             <min>0.10</min>

File: urdf/mobile_robot_macro.xacro (robot description, xacro)
@@ -73,5 +73,5 @@
         <inertial>
           <!--assign inertial properties to drive wheels -->
-          <mass value="1"/>
+          <mass value="1.5"/>
           <inertia ixx="0.1" ixy="0" ixz="0" iyy="0.1" iyz="0" izz="0.1"/>
         </inertial>
@@ -223,21 +223,21 @@
     <xacro:wheel prefix="right" reflect="-1"/>
     <gazebo reference="right_wheel">
-      <mu1>100000.0</mu1>
-      <mu2>100000.0</mu2>
+      <mu1>10000000.0</mu1>
+      <mu2>10000000.0</mu2>
       <material>Gazebo/Black</material>
     </gazebo>
     <gazebo reference="left_wheel">
-      <mu1>100000.0</mu1>
-      <mu2>100000.0</mu2>
+      <mu1>10000000.0</mu1>
+      <mu2>10000000.0</mu2>
       <material>Gazebo/Black</material>
     </gazebo>
     <gazebo reference="right_casterwheel">
-      <mu1>100000.0</mu1>
-      <mu2>100000.0</mu2>
+      <mu1>10000000.0</mu1>
+      <mu2>10000000.0</mu2>
       <material>Gazebo/Black</material>
     </gazebo>
     <gazebo reference="left_casterwheel">
-      <mu1>100000.0</mu1>
-      <mu2>100000.0</mu2>
+      <mu1>10000000.0</mu1>
+      <mu2>10000000.0</mu2>
       <material>Gazebo/Black</material>
     </gazebo>
@@ -245,6 +245,6 @@
     <gazebo>
       <plugin name="joint_state_publisher" filename="libgazebo_ros_joint_state_publisher.so">
-        <jointName>cast2bracket_right, cast2bracket_left, right_caster_joint, left_caster_joint
-        </jointName>
+        <jointName>cast2bracket_right, cast2bracket_left, right_caster_joint, left_caster_joint</jointName>
+        <updateRate>60</updateRate>
       </plugin>
     </gazebo>

File: urdf/mobile_robot_transmission.xacro (robot description, xacro)
@@ -2,5 +2,9 @@
 <robot xmlns:xacro="http://www.ros.org/wiki/xacro">
   <xacro:macro name="mobile_robot_transmission" params="prefix">
-    <xacro:arg name="use_gazebo_plugin" default="false"/>
+    <xacro:arg name="use_gazebo_plugin" default="true"/>
+    <xacro:arg name="use_transmission" default="false"/>
+    <!-- copied from robot macro-->
+    <xacro:property name="tirediam" value="0.3302"/>
+    <xacro:property name="track" value="0.53515"/>
     <xacro:if value="$(arg use_gazebo_plugin)">
       <gazebo>
@@ -19,10 +23,13 @@
           <legacyMode>false</legacyMode>
           <publishWheelTF>true</publishWheelTF>
+          <publishTf>true</publishTf>
           <publishWheelJointState>true</publishWheelJointState>
+          <wheelAcceleration>10</wheelAcceleration>
+          <wheelTorque>100</wheelTorque>
         </plugin>
       </gazebo>
     </xacro:if>
-    <xacro:unless value="$(arg use_gazebo_plugin)">
-      <transmission name="left_wheel_trans" type="SimpleTransmission">
+    <xacro:if value="$(arg use_transmission)">
+      <transmission name="left_wheel_trans">
         <type>transmission_interface/SimpleTransmission</type>
         <actuator name="left_wheel_motor">
@@ -33,5 +40,5 @@
         </joint>
       </transmission>
-      <transmission name="right_wheel_trans" type="SimpleTransmission">
+      <transmission name="right_wheel_trans">
         <type>transmission_interface/SimpleTransmission</type>
         <actuator name="right_wheel_motor">
@@ -44,9 +51,9 @@
       <gazebo>
         <plugin name="ros_control" filename="libgazebo_ros_control.so">
-          <robotNamespace></robotNamespace>
+          <!-- <robotNamespace></robotNamespace> -->
           <!-- <robotSimType>gazebo_ros_control/DefaultRobotHWSim</robotSimType> -->
         </plugin>
       </gazebo>
-    </xacro:unless>
+    </xacro:if>
   </xacro:macro>
 </robot>
