Commit message: improve robot model

File: urdf/mobile_robot.xacro (robot description, xacro)
@@ -3,5 +3,5 @@
   <xacro:include filename="$(find simple_mobile_robot)/urdf/mobile_robot_macro.xacro"/>
   <xacro:include filename="$(find simple_mobile_robot)/urdf/mobile_robot_lidar.xacro"/>
-	<xacro:include filename="$(find simple_mobile_robot)/urdf/mobile_robot_transmission.xacro" />
+  <xacro:include filename="$(find simple_mobile_robot)/urdf/mobile_robot_transmission.xacro" />
   <xacro:mobile_robot_macro prefix=""/>
   <xacro:mobile_robot_lidar prefix=""/>

File: urdf/mobile_robot_lidar.xacro (robot description, xacro)
@@ -4,5 +4,5 @@
     <!-- copied from robot macro -->
     <xacro:property name="bodylen" value="0.5461"/>
-    <xacro:property name="lidarlen" value="0.1"/>
+    <xacro:property name="lidarlen" value="0.05"/>
     <xacro:property name="lidarOZ" value="-0.03"/>
     <!-- add a simulated lidar, including visual, collision and inertial properties, and physics simulation-->

File: urdf/mobile_robot_macro.xacro (robot description, xacro)
@@ -4,8 +4,7 @@
     <!-- define the base-link origin to lie at floor level, between the drive wheels-->
     <!--main body is a simple box; origin is a center of box-->
-    <xacro:property name="bodylen" value="0.5461"/>
-    <xacro:property name="bodywidth" value="0.4572"/>
-    <xacro:property name="bodyheight" value="0.2"/>
-    <xacro:property name="bodyclearance" value="0.4"/>
+    <xacro:property name="bodylen" value="0.5061"/>
+    <xacro:property name="bodywidth" value="0.4072"/>
+    <xacro:property name="bodyheight" value="0.16"/>
     <!--clearance from bottom of box to ground-->
     <!-- derived values-->
@@ -15,5 +14,5 @@
     <xacro:property name="bodyOX" value="${-half_bodylen}"/>
     <xacro:property name="bodyOY" value="0"/>
-    <xacro:property name="bodyOZ" value="0.45"/>
+    <xacro:property name="bodyOZ" value="0.35"/>
     <!-- define the drive-wheel dimensions-->
     <xacro:property name="tirediam" value="0.3302"/>
@@ -21,9 +20,9 @@
     <xacro:property name="tirewidth" value="0.06985"/>
     <!-- "track" is the distance between the drive wheels -->
-    <xacro:property name="track" value="0.53515"/>
+    <xacro:property name="track" value="0.51015"/>
     <xacro:property name="M_PI" value="3.1415926535897931"/>
     <xacro:property name="boschwidth" value="0.0381"/>
-    <xacro:property name="casterdrop" value="0.125"/>
-    <xacro:property name="frontdrop" value="${tirerad+0.02}"/>
+    <xacro:property name="casterdrop" value="0.05"/>
+    <xacro:property name="frontdrop" value="${tirerad+0.02-0.1}"/>
     <xacro:property name="bracketwidth" value="0.1175"/>
     <xacro:property name="bracketheight" value="0.16"/>
@@ -53,5 +52,5 @@
           <origin xyz="0 0 0" rpy="0 0 0"/>
         </collision>
-        <xacro:default_inertial mass="0.25"/>
+        <xacro:default_inertial mass="0.2"/>
       </link>
       <joint name="hoop2base_${prefix}" type="fixed">
@@ -82,5 +81,5 @@
         <child link="${prefix}_wheel"/>
         <origin xyz="0 ${reflect*track/2} ${tirerad}" rpy="0 ${M_PI/2} ${M_PI/2}"/>
-        <limit effort="100" velocity="15"/>
+        <limit effort="100" velocity="25"/>
         <joint_properties damping="0.0" friction="0.0"/>
       </joint>
@@ -120,5 +119,5 @@
           <origin xyz="0 0 0" rpy="0 0 0"/>
         </collision>
-        <xacro:default_inertial mass="0.2"/>
+        <xacro:default_inertial mass="0.1"/>
       </link>
       <joint name="cast2bracket_${prefix}" type="continuous">
@@ -142,5 +141,5 @@
           <origin xyz="0 0 0" rpy="${M_PI/2} ${-bracketangle} ${M_PI/2}"/>
         </collision>
-        <xacro:default_inertial mass="0.2"/>
+        <xacro:default_inertial mass="0.05"/>
       </link>
       <joint name="brack2top1_${prefix}" type="fixed">
@@ -162,5 +161,5 @@
           <origin xyz="0 0 0" rpy="${M_PI/2} ${-bracketangle} ${M_PI/2}"/>
         </collision>
-        <xacro:default_inertial mass="0.2"/>
+        <xacro:default_inertial mass="0.05"/>
       </link>
       <joint name="brack2top2_${prefix}" type="fixed">
@@ -181,5 +180,5 @@
         </collision>
         <!-- accept default inertial properties for caster wheels-->
-        <xacro:default_inertial mass="0.5"/>
+        <xacro:default_inertial mass="0.3"/>
       </link>
       <joint name="${prefix}_caster_joint" type="continuous">
@@ -188,5 +187,5 @@
         <child link="${prefix}_casterwheel"/>
         <origin xyz="${-casterwidth/2-.02} .053 -.053" rpy="0 ${M_PI/2} 0"/>
-        <limit effort="100" velocity="15"/>
+        <limit effort="100" velocity="25"/>
         <joint_properties damping="0.0" friction="0.0"/>
       </joint>
@@ -205,9 +204,5 @@
         <origin xyz="0 0 0" rpy="0 0 0"/>
       </collision>
-      <inertial>
-        <!--assign almost all the mass to the main body box; set m= 100kg; treat I as approx m*r^2 -->
-        <mass value="100"/>
-        <inertia ixx="10" ixy="0" ixz="0" iyy="10" iyz="0" izz="10"/>
-      </inertial>
+      <xacro:default_inertial mass="100"/>
     </link>
     <!-- Base link is the footprint of the robot -->
@@ -218,8 +213,9 @@
       <child link="robot_body"/>
     </joint>
-    <xacro:caster prefix="left" reflect="1"/>
-    <xacro:caster prefix="right" reflect="-1"/>
+    <!-- <xacro:caster prefix="left" reflect="1"/> -->
+    <!-- <xacro:caster prefix="right" reflect="-1"/> -->
     <xacro:wheel prefix="left" reflect="1"/>
     <xacro:wheel prefix="right" reflect="-1"/>
+    <xacro:caster prefix="rear" reflect="0"/>
     <gazebo reference="right_wheel">
       <mu1>100000.0</mu1>
@@ -232,15 +228,26 @@
       <material>Gazebo/Black</material>
     </gazebo>
-    <gazebo reference="right_casterwheel">
-      <mu1>100000.0</mu1>
-      <mu2>100000.0</mu2>
+    <gazebo reference="rear_casterwheel">
+      <mu1>1000.0</mu1>
+      <mu2>1000.0</mu2>
+      <material>Gazebo/Black</material>
+    </gazebo>
+    <gazebo>
+      <plugin name="joint_state_publisher" filename="libgazebo_ros_joint_state_publisher.so">
+        <jointName>rear_caster_joint</jointName>
+        <updateRate>60</updateRate>
+      </plugin>
+    </gazebo>
+<!--
+     <gazebo reference="right_casterwheel">
+      <mu1>1000.0</mu1>
+      <mu2>1000.0</mu2>
       <material>Gazebo/Black</material>
     </gazebo>
     <gazebo reference="left_casterwheel">
-      <mu1>100000.0</mu1>
-      <mu2>100000.0</mu2>
-      <material>Gazebo/Black</material>
-    </gazebo>
-    <!-- publish joint state for passive wheels -->
+      <mu1>1000.0</mu1>
+      <mu2>1000.0</mu2>
+      <material>Gazebo/Black</material>
+    </gazebo>
     <gazebo>
       <plugin name="joint_state_publisher" filename="libgazebo_ros_joint_state_publisher.so">
@@ -248,5 +255,6 @@
         <updateRate>60</updateRate>
       </plugin>
-    </gazebo>
+    </gazebo> -->
+    <!-- publish joint state for passive wheels -->
   </xacro:macro>
 </robot>

File: urdf/mobile_robot_transmission.xacro (robot description, xacro)
@@ -25,5 +25,5 @@
           <publishTf>true</publishTf>
           <publishWheelJointState>true</publishWheelJointState>
-          <wheelAcceleration>10</wheelAcceleration>
+          <wheelAcceleration>40</wheelAcceleration>
           <wheelTorque>100</wheelTorque>
         </plugin>
